File: input-power.brd (EAGLE design)
At the start: 100 x 80 mm, 13 parts, among them J1 Battery, J2 Solar

Commit message: Work on power board
Parts:
- removed TP1, TP2, TP4: TPSB1,27, testpad:B1,27
- added D4: (no value), diode:SMB
- added J3: Battery, SparkFun-Connectors:1X02_LONGPADS
- added LED1: GREEN, led:LED3MM
- added R1: 1M, resistor:R0805
- added R3: 3K3, resistor:R0805
- added TP5: TPSB1,27, testpad:B1,27
- added U$3: 2A, fuse:MF-SMDF050
- added U$6: XL6009_BOOST_MODULE, breakout-modules:XL6009_BOOST_MODULE
- added U$9: FDS6675, Semiconductors:SO08
- moved U$10 17.2 mm to (14.0, 64.0), turned to 180 degrees
- moved J2 9.00 mm to (6.00, 60.0)
- moved D2 4.47 mm to (24.0, 64.0), turned to 180 degrees
- moved J1 3.51 mm to (9.00, 40.0)
Connections:
- new net BT_POWER_ENABLE: R1.2, TP5.TP, U$9.4
- new net N$6: D4.C, U$3.1, U$6.V_OUT
- new net N$9: LED1.K, R3.1
- new net VALVE: J3.1, U$3.2
- new net V_VALVE_UNREG: LED1.A, U$6.V_IN, U$9.5, U$9.6, U$9.7, U$9.8
- net GND: now also D4.A, J3.2, R3.2, U$6.V_IN_GND, U$6.V_OUT_GND; no longer TP4.TP
- net V_CHARGER: no longer TP1.TP
- net V_UNREG: now also R1.1, U$9.1, U$9.2, U$9.3; no longer TP2.TP
Routing:
- net V_VALVE_UNREG: track 0.00 -> 63.2 mm
- net BT_POWER_ENABLE: track 0.00 -> 29.2 mm
- net N$6: track 0.00 -> 16.4 mm
- net V_SOLAR: track 24.2 -> 10.9 mm
- net V_UNREG: track 38.4 -> 50.3 mm
- net VALVE: track 0.00 -> 7.64 mm
- net V_SOLAR_FUSED: track 21.0 -> 16.8 mm
- net N$9: track 0.00 -> 4.12 mm
- net N$3: track 17.6 -> 14.7 mm
Other:
- board size 100 x 80 mm -> 65 x 80 mm
