File: input-power.sch (EAGLE design)
At the start: 13 parts, among them J1 Battery, J2 Solar

Commit message: Work on power board
Parts:
- removed TP1, TP2, TP4: TPSB1,27, testpad:TPSB1,27
- added D4: (no value), diode:DIODE-SMB
- added J3: Battery, SparkFun-Connectors:M02PTH3
- added LED1: GREEN, led:LED3MM
- added R1: 1M, resistor:R-EU_R0805
- added R3: 3K3, resistor:R-EU_R0805
- added TP5: TPSB1,27, testpad:TPSB1,27
- added U$3: 2A, fuse:MF-SMDF150
- added U$6: XL6009_BOOST_MODULE, breakout-modules:XL6009_BOOST_MODULE
- added U$9: FDS6675, Semiconductors:FDS6675
Connections:
- new net BT_POWER_ENABLE: R1.2, TP5.PP, U$9.G
- new net N$6: D4.C, U$3.1, U$6.V_OUT
- new net N$9: LED1.C, R3.1
- new net VALVE: J3.1, U$3.2
- new net V_VALVE_UNREG: LED1.A, U$6.V_IN, U$9.D
- net GND: now also D4.A, J3.2, R3.2, U$6.V_IN_GND, U$6.V_OUT_GND; no longer TP4.PP
- net V_CHARGER: no longer TP1.PP
- net V_UNREG: now also R1.1, U$9.S; no longer TP2.PP
Other:
- note added: "Valve power"
- moved on the sheet: D3
