File: Vattenkran.sch (EAGLE design)
At the start: 13 parts, among them Q2 32KHz

Commit message: Replaced crystal
Parts:
- removed Q2: 32KHz, adafruit:CRYSTALTC38H
- added U$2: 32Khz, Semiconductors:CLOCK_CRYSTAL_32KHZ
Connections:
- net N$4: now also U$2.P$1; no longer Q2.2
- net N$5: now also U$2.P$2; no longer Q2.1
Changed lines of the file:
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@@
 <part name="U$1" library="adafruit" deviceset="DS1302" device=""/>
 <part name="SUPPLY9" library="supply2" library_urn="urn:adsk.eagle:library:372" deviceset="GND" device=""/>
-<part name="Q2" library="adafruit" deviceset="CRYSTAL" device="TC38H" value="32KHz"/>
 <part name="SUPERCAP" library="rcl" library_urn="urn:adsk.eagle:library:334" deviceset="CPOL-US" device="ETR2" package3d_urn="urn:adsk.eagle:package:23315/1" value="1F"/>
 <part name="SUPPLY10" library="supply2" library_urn="urn:adsk.eagle:library:372" deviceset="GND" device=""/>
@@
 <part name="TP2" library="testpad" library_urn="urn:adsk.eagle:library:385" deviceset="TP" device="B1,27" package3d_urn="urn:adsk.eagle:package:27944/1"/>
 <part name="TP3" library="testpad" library_urn="urn:adsk.eagle:library:385" deviceset="TP" device="B1,27" package3d_urn="urn:adsk.eagle:package:27944/1"/>
+<part name="U$2" library="Semiconductors" deviceset="CLOCK_CRYSTAL_32KHZ" device="" value="32Khz"/>
 </parts>
 <sheets>
@@
 <instance part="U$1" gate="G$1" x="116.84" y="12.7"/>
 <instance part="SUPPLY9" gate="GND" x="116.84" y="-5.08"/>
-<instance part="Q2" gate="G$1" x="114.3" y="35.56" rot="R180"/>
 <instance part="SUPERCAP" gate="G$1" x="134.62" y="5.08"/>
 <instance part="SUPPLY10" gate="GND" x="134.62" y="-2.54"/>
@@
 <instance part="TP2" gate="G$1" x="38.1" y="10.16" rot="R270"/>
 <instance part="TP3" gate="G$1" x="-15.24" y="17.78" rot="R90"/>
+<instance part="U$2" gate="G$1" x="114.3" y="48.26"/>
 </instances>
 <busses>
@@
 <net name="N$4" class="0">
 <segment>
-<pinref part="Q2" gate="G$1" pin="2"/>
 <pinref part="U$1" gate="G$1" pin="X1"/>
 <wire x1="111.76" y1="35.56" x2="111.76" y2="27.94" width="0.1524" layer="91"/>
+<pinref part="U$2" gate="G$1" pin="P$1"/>
+<wire x1="104.14" y1="48.26" x2="104.14" y2="35.56" width="0.1524" layer="91"/>
+<wire x1="104.14" y1="35.56" x2="111.76" y2="35.56" width="0.1524" layer="91"/>
 </segment>
 </net>
@@
 <segment>
 <pinref part="U$1" gate="G$1" pin="X2"/>
-<pinref part="Q2" gate="G$1" pin="1"/>
 <wire x1="116.84" y1="27.94" x2="116.84" y2="35.56" width="0.1524" layer="91"/>
-</segment>
-</net>
+<pinref part="U$2" gate="G$1" pin="P$2"/>
+<wire x1="124.46" y1="48.26" x2="124.46" y2="35.56" width="0.1524" layer="91"/>
+<wire x1="124.46" y1="35.56" x2="116.84" y2="35.56" width="0.1524" layer="91"/>
+</segment>
+</net>

Commit message: Added cap
Parts:
- added C4: 100µF, resistor:CPOL-USD
Connections:
- net GND: now also C4.-
- net VCC5: now also C4.+
Other:
- moved on the sheet: C1, C3, SUPERCAP, U$1, U$2
Changed lines of the file:
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@@
 <part name="TP3" library="testpad" library_urn="urn:adsk.eagle:library:385" deviceset="TP" device="B1,27" package3d_urn="urn:adsk.eagle:package:27944/1"/>
 <part name="U$2" library="Semiconductors" deviceset="CLOCK_CRYSTAL_32KHZ" device="" value="32Khz"/>
+<part name="C4" library="resistor" library_urn="urn:adsk.eagle:library:348" deviceset="CPOL-US" device="D" package3d_urn="urn:adsk.eagle:package:25914/1" value="100µF"/>
+<part name="SUPPLY1" library="supply2" library_urn="urn:adsk.eagle:library:372" deviceset="GND" device=""/>
 </parts>
 <sheets>
 <sheet>
 <plain>
-<text x="78.74" y="33.02" size="1.778" layer="91">Real time clock</text>
+<text x="119.38" y="22.86" size="1.778" layer="91">Real time clock</text>
 <text x="33.02" y="-38.1" size="1.778" layer="91">Bluetooth</text>
 </plain>
 <instances>
-<instance part="U$1" gate="G$1" x="116.84" y="12.7"/>
-<instance part="SUPPLY9" gate="GND" x="116.84" y="-5.08"/>
-<instance part="SUPERCAP" gate="G$1" x="134.62" y="5.08"/>
-<instance part="SUPPLY10" gate="GND" x="134.62" y="-2.54"/>
+<instance part="U$1" gate="G$1" x="157.48" y="2.54"/>
+<instance part="SUPPLY9" gate="GND" x="157.48" y="-15.24"/>
+<instance part="SUPERCAP" gate="G$1" x="175.26" y="-5.08"/>
+<instance part="SUPPLY10" gate="GND" x="175.26" y="-12.7"/>
 <instance part="U$4" gate="G$1" x="71.12" y="-60.96"/>
 <instance part="U$7" gate="G$1" x="15.24" y="15.24"/>
@@
 <instance part="LED2" gate="G$1" x="132.08" y="-60.96"/>
 <instance part="SUPPLY20" gate="GND" x="132.08" y="-83.82"/>
-<instance part="C1" gate="G$1" x="154.94" y="15.24"/>
+<instance part="C1" gate="G$1" x="195.58" y="5.08"/>
 <instance part="C2" gate="G$1" x="78.74" y="-43.18" rot="R90"/>
-<instance part="C3" gate="G$1" x="55.88" y="27.94" rot="R90"/>
-<instance part="SUPPLY21" gate="GND" x="154.94" y="7.62"/>
-<instance part="SUPPLY22" gate="GND" x="66.04" y="27.94" rot="R90"/>
+<instance part="C3" gate="G$1" x="83.82" y="22.86"/>
+<instance part="SUPPLY21" gate="GND" x="195.58" y="-2.54"/>
+<instance part="SUPPLY22" gate="GND" x="83.82" y="10.16"/>
 <instance part="SUPPLY23" gate="GND" x="91.44" y="-45.72"/>
 <instance part="TP1" gate="G$1" x="38.1" y="40.64"/>
 <instance part="TP2" gate="G$1" x="38.1" y="10.16" rot="R270"/>
 <instance part="TP3" gate="G$1" x="-15.24" y="17.78" rot="R90"/>
-<instance part="U$2" gate="G$1" x="114.3" y="48.26"/>
+<instance part="U$2" gate="G$1" x="154.94" y="38.1"/>
+<instance part="C4" gate="G$1" x="73.66" y="22.86"/>
+<instance part="SUPPLY1" gate="GND" x="73.66" y="10.16"/>
 </instances>
 <busses>
@@
 <pinref part="C3" gate="G$1" pin="2"/>
 <pinref part="SUPPLY22" gate="GND" pin="GND"/>
-<wire x1="60.96" y1="27.94" x2="63.5" y2="27.94" width="0.1524" layer="91"/>
+<wire x1="83.82" y1="17.78" x2="83.82" y2="12.7" width="0.1524" layer="91"/>
 </segment>
 <segment>
@@
 <wire x1="83.82" y1="-43.18" x2="91.44" y2="-43.18" width="0.1524" layer="91"/>
 <pinref part="C2" gate="G$1" pin="2"/>
+</segment>
+<segment>
+<pinref part="C4" gate="G$1" pin="-"/>
+<pinref part="SUPPLY1" gate="GND" pin="GND"/>
+<wire x1="73.66" y1="12.7" x2="73.66" y2="17.78" width="0.1524" layer="91"/>
 </segment>
 </net>
@@
 <segment>
 <pinref part="U$1" gate="G$1" pin="CE"/>
-<junction x="101.6" y="15.24"/>
-<wire x1="101.6" y1="15.24" x2="93.98" y2="15.24" width="0.1524" layer="91"/>
-<label x="78.74" y="15.24" size="1.778" layer="95"/>
+<junction x="142.24" y="5.08"/>
+<wire x1="142.24" y1="5.08" x2="134.62" y2="5.08" width="0.1524" layer="91"/>
+<label x="119.38" y="5.08" size="1.778" layer="95"/>
 </segment>
 <segment>
@@
 <segment>
 <pinref part="U$1" gate="G$1" pin="I/O"/>
-<junction x="101.6" y="12.7"/>
-<wire x1="101.6" y1="12.7" x2="93.98" y2="12.7" width="0.1524" layer="91"/>
-<label x="78.74" y="12.7" size="1.778" layer="95"/>
+<junction x="142.24" y="2.54"/>
+<wire x1="142.24" y1="2.54" x2="134.62" y2="2.54" width="0.1524" layer="91"/>
+<label x="119.38" y="2.54" size="1.778" layer="95"/>
 </segment>
 <segment>
@@
 <segment>
 <pinref part="U$1" gate="G$1" pin="SCLK"/>
-<junction x="101.6" y="10.16"/>
-<wire x1="101.6" y1="10.16" x2="93.98" y2="10.16" width="0.1524" layer="91"/>
-<label x="78.74" y="10.16" size="1.778" layer="95"/>
+<junction x="142.24" y="0"/>
+<wire x1="142.24" y1="0" x2="134.62" y2="0" width="0.1524" layer="91"/>
+<label x="119.38" y="0" size="1.778" layer="95"/>
 </segment>
 <segment>
@@
 <pinref part="U$1" gate="G$1" pin="VBAT"/>
 <pinref part="SUPERCAP" gate="G$1" pin="+"/>
-<wire x1="132.08" y1="10.16" x2="134.62" y2="10.16" width="0.1524" layer="91"/>
-<wire x1="134.62" y1="10.16" x2="134.62" y2="7.62" width="0.1524" layer="91"/>
-<junction x="132.08" y="10.16"/>
+<wire x1="172.72" y1="0" x2="175.26" y2="0" width="0.1524" layer="91"/>
+<wire x1="175.26" y1="0" x2="175.26" y2="-2.54" width="0.1524" layer="91"/>
+<junction x="172.72" y="0"/>
 </segment>
 </net>
@@
 <junction x="38.1" y="38.1"/>
 <pinref part="C3" gate="G$1" pin="1"/>
-<wire x1="38.1" y1="27.94" x2="53.34" y2="27.94" width="0.1524" layer="91"/>
+<wire x1="38.1" y1="27.94" x2="73.66" y2="27.94" width="0.1524" layer="91"/>
 <junction x="38.1" y="27.94"/>
+<pinref part="C4" gate="G$1" pin="+"/>
+<wire x1="73.66" y1="27.94" x2="83.82" y2="27.94" width="0.1524" layer="91"/>
+<wire x1="83.82" y1="27.94" x2="83.82" y2="25.4" width="0.1524" layer="91"/>
+<wire x1="73.66" y1="25.4" x2="73.66" y2="27.94" width="0.1524" layer="91"/>
+<junction x="73.66" y="27.94"/>
 </segment>
 </net>
 <net name="VCC33" class="0">
 <segment>
-<label x="134.62" y="20.32" size="1.778" layer="95"/>
+<label x="175.26" y="10.16" size="1.778" layer="95"/>
 <pinref part="U$1" gate="G$1" pin="VCC"/>
-<wire x1="132.08" y1="17.78" x2="154.94" y2="17.78" width="0.1524" layer="91"/>
-<junction x="132.08" y="17.78"/>
+<wire x1="172.72" y1="7.62" x2="195.58" y2="7.62" width="0.1524" layer="91"/>
+<junction x="172.72" y="7.62"/>
 <pinref part="C1" gate="G$1" pin="1"/>
 </segment>
@@
 <segment>
 <pinref part="U$1" gate="G$1" pin="X1"/>
-<wire x1="111.76" y1="35.56" x2="111.76" y2="27.94" width="0.1524" layer="91"/>
+<wire x1="152.4" y1="25.4" x2="152.4" y2="17.78" width="0.1524" layer="91"/>
 <pinref part="U$2" gate="G$1" pin="P$1"/>
-<wire x1="104.14" y1="48.26" x2="104.14" y2="35.56" width="0.1524" layer="91"/>
-<wire x1="104.14" y1="35.56" x2="111.76" y2="35.56" width="0.1524" layer="91"/>
+<wire x1="144.78" y1="38.1" x2="144.78" y2="25.4" width="0.1524" layer="91"/>
+<wire x1="144.78" y1="25.4" x2="152.4" y2="25.4" width="0.1524" layer="91"/>
 </segment>
 </net>
@@
 <segment>
 <pinref part="U$1" gate="G$1" pin="X2"/>
-<wire x1="116.84" y1="27.94" x2="116.84" y2="35.56" width="0.1524" layer="91"/>
+<wire x1="157.48" y1="17.78" x2="157.48" y2="25.4" width="0.1524" layer="91"/>
 <pinref part="U$2" gate="G$1" pin="P$2"/>
-<wire x1="124.46" y1="48.26" x2="124.46" y2="35.56" width="0.1524" layer="91"/>
-<wire x1="124.46" y1="35.56" x2="116.84" y2="35.56" width="0.1524" layer="91"/>
-</segment>
-</net>
+<wire x1="165.1" y1="38.1" x2="165.1" y2="25.4" width="0.1524" layer="91"/>
+<wire x1="165.1" y1="25.4" x2="157.48" y2="25.4" width="0.1524" layer="91"/>
+</segment>
+</net>
